File: Diplomka/MainBoard.brd (EAGLE design)
At the start: 100 x 100 mm, 44 parts, among them K1 ARK550/2, Q1 AP2012P3C-P22, Q2 BC817-40LT1SMD, Q3 SS8050-G, Q4 SS8050-G, U1 ESP32-WROOM-32, U2 AMS1117-3.3

Commit message: Design hotový, čas importovat bitmapu.
Parts:
- moved U$4 1.00 mm to (50.0, 18.0)
Routing:
- net CTS: track 64.2 -> 65.6 mm
- net 5V: track 134.8 -> 134.1 mm
Other:
- board text added: "CTS"
- board text added: "Created at VSB By Alexander Barsc And Radim Hercik"
- board text added: "DTR"
- board text added: "GND"
- board text added: "RX"
- board text added: "TX"
- board text added: "VCC"
- board text added: "VIN"
