File: Diplomka/MainBoard.sch (EAGLE design)
At the start: 44 parts, among them K1 ARK550/2, Q1 PT15-21C/TR8, Q2 SS8050-G, Q3 SS8050-G, Q4 SS8050-G, U1 ESP32-WROOM-32, U2 AMS1117-3.3

Commit message: WIP
Parts:
- R1, R4: value 1K -> 100K
- R3, R5: value 2K -> 200K
Other:
- note added: "Nahrazen fotorezistorem o hodnote 5 - 10K pri svetle"
- note added: "PHOTOTRAN_CONTROL je nutne premistit na pin co slouzi jako vystup"
